Commit message: gym env upgrades

File: assets/kitchen_knife/kitchen_knife.urdf (robot description, URDF)
Before this commit: robot sharp_knife, 1 links, 0 joints
Links:
- link baseLink: geometry collision mesh filename=sharp_knife.obj scale=0.001 0.001 0.001; visual mesh filename=sharp_knife.obj scale=0.001 0.001 0.001

File: assets/spatula/spatula.urdf (robot description, URDF)
Before this commit: robot spatula, 1 links, 0 joints
Links:
- link baseLink: geometry collision mesh filename=spatula.obj scale=0.01 0.01 0.01; visual mesh filename=spatula.obj scale=0.01 0.01 0.01

File: assets/spoon/spoon.urdf (robot description, URDF)
Before this commit: robot spoon, 1 links, 0 joints
Links:
- link baseLink: geometry collision mesh filename=spoon.obj scale=0.001 0.001 0.001; visual mesh filename=spoon.obj scale=0.001 0.001 0.001
